File: projects/CarBatteryCharger/Caricabatteria 1.0.brd (EAGLE design)
At the start: 50.5 x 61 mm, 22 parts, among them IC1 7912, T1 TAG 665-100, X1 MKDSN1,5/2-5,08, X2 MKDSN1,5/2-5,08, X3 MKDSN1,5/2-5,08

Commit message: Tweak of PCB
Tweak of PCB
Parts:
- removed X2, X3: MKDSN1,5/2-5,08, con-phoenix-508-IZ0VLL:MKDSN1,5/2-5,08
- added AMP, BATT-VOLT: MKDSN1,5/2-5,08, con-phoenix-508-IZ0VLL:MKDSN1,5/2-5,08
- moved R6 1.80 mm to (41.9, 48.3)
- moved C2 1.27 mm to (31.8, 11.4)
- moved R5 1.27 mm to (38.1, 40.6)
- renumbered X1 to 13.5VAC
Connections:
- net N$11: now also AMP.1; no longer X2.1
- net N$3: now also AMP.2, BATT-VOLT.1; no longer X2.2, X3.1
- net N$8: now also BATT-VOLT.2; no longer X3.2
Routing:
- net N$11: track 98.8 -> 96.3 mm
- net N$8: track 55.5 -> 53.4 mm
- net N$3: track 38.1 -> 36.7 mm
- net N$7: track 95.7 -> 94.4 mm
- net N$9: track 15.2 -> 14.5 mm
- net N$10: track 5.61 -> 6.13 mm
Other:
- board text added: "AC IN * 13.5V"
- board text added: "AMPEROMETRO"
- board text added: "BATT-VOLT"
- board text added: "CARICABATTERIA AUTO ARI VIGEVANO"
- board text added: "Salvatore Mele, IZ0VLL"
